File: hardware-electronics/M2SmartHome/M2SmartHome.kicad_pcb (KiCad board)
At the start: 2 copper layers, 0 parts

Commit message: Created basic mechanical mockup of the device
Parts:
- added M1: M.2-B-KEY-2280-ADAPTER, footprints:M.2-B-KEY-2280-ADAPTER, F.Cu at (90.8, 165.0)
- added REF**: QFN-20-1EP_3x3mm_P0.4mm_EP1.65x1.65mm, Package_DFN_QFN:QFN-20-1EP_3x3mm_P0.4mm_EP1.65x1.65mm, F.Cu at (97.9, 76.5)
- added REF**: QFN-20-1EP_3x3mm_P0.4mm_EP1.65x1.65mm, Package_DFN_QFN:QFN-20-1EP_3x3mm_P0.4mm_EP1.65x1.65mm, F.Cu at (95.5, 87.4)
- added REF**: QFN-32-1EP_4x4mm_P0.4mm_EP2.9x2.9mm, Package_DFN_QFN:QFN-32-1EP_4x4mm_P0.4mm_EP2.9x2.9mm, F.Cu at (84.3, 87.1)
- added REF**: QFN-32-1EP_4x4mm_P0.4mm_EP2.9x2.9mm, Package_DFN_QFN:QFN-32-1EP_4x4mm_P0.4mm_EP2.9x2.9mm, F.Cu at (84.6, 77.3)
- added REF**: microSD_HC_Hirose_DM3AT-SF-PEJM5, Connector_Card:microSD_HC_Hirose_DM3AT-SF-PEJM5, F.Cu at (88.1, 99.1)
- added REF**: VQFN-64-1EP_9x9mm_P0.5mm_EP5.4x5.4mm, Package_DFN_QFN:VQFN-64-1EP_9x9mm_P0.5mm_EP5.4x5.4mm, F.Cu at (88.8, 131.8)
- added U1: EMMC08G-ML36-01B00, footprints:BGA153N50P14X14_1300X1150X100N, F.Cu at (89.9, 116.7)
- added U2: PI7C9X440SLBFDE, footprints:QFP40P1600X1600X160-129N, F.Cu at (91.2, 149.6)
Other:
- board outline added: 24 x 95 mm
