File: hardware-electronics/z-wave.kicad_sch (KiCad schematic)
At the start: 2 parts, among them U4 CP2102N-A02-GQFN20, U6 EFR32ZG14P231F256GM32-BR

Commit message: SCH WIP Z-wave
Parts:
- added C1: C_100n_0603, C_100n_0603:C_0603_1608Metric, symbol C_100n_0603:C_100n_0603
- added C2, C3, C4, C5: C_4u7_6.3V_0402, C_4u7_6.3V_0402:C_0402_1005Metric, symbol C_4u7_6.3V_0402:C_4u7_6.3V_0402
- added C6, C7: GRM1555C1H1R9WA01D, GRM1555C1H1R9WA01D:CAPC1005X55N, symbol M2SmartHomeSymbols:GRM1555C1H1R9WA01D
- added L1: L_4u7_0.4A_0805, L_4u7_0.4A_0805:L_0805_2012Metric, symbol L_4u7_0.4A_0805:L_4u7_0.4A_0805
- added L2: LQW15AN18NJ00D, LQW15AN18NJ00D:INDC1006X60N, symbol M2SmartHomeSymbols:LQW15AN18NJ00D
- added L3, L4: LQW15AN3N3B80D, LQW15AN3N3B80D:INDC1006X60N, symbol M2SmartHomeSymbols:LQW15AN3N3B80D
- added U9: 0900BL15C050E, 0900BL15C050E:XCVR_0900BL15C050E, symbol M2SmartHomeSymbols:0900BL15C050E
Connections:
- net at U6.11 (SUBGRF_IP): now also C7.1, L2.2
- net at U6.12 (SUBGRF_IN): now also C6.1, L2.1
- net GND: now reaches U6.13 (RFVSS)
- net GND: now also U6.25 (VREGVSS), C1.1, C2.1, C3.1, C4.1, C5.1
- net +3.3V: now reaches U6.22 (AVDD)
- net +3.3V: now also U6.27 (VREGVDD), U6.30 (IOVDD)
- net at U6.26 (VREGSW): now also L1.1
- net at U6.28 (DVDD): now also U6.5 (RFVDD), C2.2, C3.2, C4.2, C5.2, L1.2
- net at U6.29 (DECOUPLE): now also C1.2
- new net: C7.2, L4.1
- new net: C6.2, L3.1
Other:
- note added: "where pin 10?"
- moved on the sheet: U6

Commit message: SCH WIP z-wave
Parts:
- added C10, C8: GRM1555C1H3R3CA01D, GRM1555C1H3R3CA01D:CAPC1005X55N, symbol M2SmartHomeSymbols:GRM1555C1H3R3CA01D
- added C11: GRM155R61C224MA12D, GRM155R61C224MA12D:CAPC1005X55N, symbol M2SmartHomeSymbols:GRM155R61C224MA12D
- added C12: GRM1555C2A560GA01D, GRM1555C2A560GA01D:INDC1005X45, symbol M2SmartHomeSymbols:GRM1555C2A560GA01D
- added C9: GRM1555C1H5R6BA01D, GRM1555C1H5R6BA01D:CAPC1005X55N, symbol M2SmartHomeSymbols:GRM1555C1H5R6BA01D
- added FL1: BLM18AG601SN1, BLM18AG601SN1:BEADC1608X95N, symbol M2SmartHomeSymbols:BLM18AG601SN1
- added J3: CONUFL001-SMD-T, CONUFL001-SMD-T:LINX_CONUFL001-SMD-T, symbol M2SmartHomeSymbols:CONUFL001-SMD-T
- added L5, L6: LQW15AN10NG00D, LQW15AN10NG00D:INDC1006X60N, symbol M2SmartHomeSymbols:LQW15AN10NG00D
Connections:
- net GND: now also U9.5 (GND), C10.1, C11.1, C12.1, C8.1, C9.1, J3.2, J3.3
- net at L4.2: now also U9.4 (BALANCED_PORT(OUT1))
- net at L3.2: now also U9.3 (BALANCED_PORT(OUT2))
- net at U9.1 (UNBALANCED_PORT(IN)): now also C8.2, L5.1
- net at U9.2 (GND/DC_FEED+RF_GND): now also C11.2, FL1.1
- new net: C9.2, L5.2, L6.1
- new net: C10.2, J3.1, L6.2
Other:
- moved on the sheet: U9
