File: hardware-electronics/wifi.kicad_sch (KiCad schematic)
At the start: 22 parts, among them J4 CONMHF1-SMD-T, U1 RTL8188FTV-VC-CG, Y5 ABM8-40.000MHZ-B2-T

Commit message: SCH fill info box
Other:
- title: (none) -> M2SmartHome
Changed lines of the file:
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@@
 	(generator_version "8.0")
 	(paper "A4")
+	(title_block
+		(title "M2SmartHome")
+		(date "2024-10-11")
+		(rev "Rev 1.0.0")
+	)
 	(junction
 		(at 200.66 93.98)

Commit message: SCH update all symbols
Parts:
- C55, C57, C75, C77: footprint C_1uF_0402:C_0402_1005Metric -> M2SmartHomeFootprints:C_0201
- C56, C58, C76, C78: footprint C_100n_0402:C_0402_1005Metric -> M2SmartHomeFootprints:C_0402
- C59: footprint C_0p9_0201:C_0201_0603Metric -> M2SmartHomeFootprints:C_0201
- C60: footprint C_1p9_0201:C_0201_0603Metric -> M2SmartHomeFootprints:C_0201
- FB8: footprint FB_120R_0603:FB_0603_1608Metric -> M2SmartHomeFootprints:FB_0603
- J4: footprint CONMHF1-SMD-T:LINX_CONMHF1-SMD-T -> M2SmartHomeFootprints:CONMHF1-SMD-T
- R38: footprint R_500R_0402:R_0402_1005Metric -> M2SmartHomeFootprints:R_0402
- R41: footprint R_24k_0402:R_0402_1005Metric -> M2SmartHomeFootprints:R_0402
- R42, R43: footprint R_10k_0402:R_0402_1005Metric -> M2SmartHomeFootprints:R_0402
- U1: footprint RTL8188FTV-VC-CG -> M2SmartHomeFootprints:RTL8188FTV-VC-CG
- Y5: footprint ABM8-40.000MHZ-B2-T -> M2SmartHomeFootprints:ABM8-40.000MHZ-B2-T
Changed lines of the file:
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@@
 			)
 		)
-		(property "Footprint" "ABM8-40.000MHZ-B2-T"
+		(property "Footprint" "M2SmartHomeFootprints:ABM8-40.000MHZ-B2-T"
 			(at 140.97 156.21 0)
 			(effects
@@
 			)
 		)
-		(property "Footprint" "FB_120R_0603:FB_0603_1608Metric"
+		(property "Footprint" "M2SmartHomeFootprints:FB_0603"
 			(at 224.79 67.31 0)
 			(effects
@@
 			)
 		)
-		(property "Footprint" "R_10k_0402:R_0402_1005Metric"
+		(property "Footprint" "M2SmartHomeFootprints:R_0402"
 			(at 215.9 71.12 0)
 			(effects
@@
 			)
 		)
-		(property "Footprint" "C_100n_0402:C_0402_1005Metric"
+		(property "Footprint" "M2SmartHomeFootprints:C_0402"
 			(at 276.86 41.91 0)
 			(effects
@@
 			)
 		)
-		(property "Footprint" "C_0p9_0201:C_0201_0603Metric"
+		(property "Footprint" "M2SmartHomeFootprints:C_0201"
 			(at 213.36 97.79 0)
 			(effects
@@
 			)
 		)
-		(property "Footprint" "C_1p9_0201:C_0201_0603Metric"
+		(property "Footprint" "M2SmartHomeFootprints:C_0201"
 			(at 199.39 97.79 0)
 			(effects
@@
 			)
 		)
-		(property "Footprint" "RTL8188FTV-VC-CG"
+		(property "Footprint" "M2SmartHomeFootprints:RTL8188FTV-VC-CG"
 			(at 144.78 96.52 0)
 			(effects
@@
 			)
 		)
-		(property "Footprint" "C_1uF_0402:C_0402_1005Metric"
+		(property "Footprint" "M2SmartHomeFootprints:C_0201"
 			(at 163.83 78.74 0)
 			(effects
@@
 			)
 		)
-		(property "Footprint" "C_1uF_0402:C_0402_1005Metric"
+		(property "Footprint" "M2SmartHomeFootprints:C_0201"
 			(at 246.38 41.91 0)
 			(effects
@@
 			)
 		)
-		(property "Footprint" "C_100n_0402:C_0402_1005Metric"
+		(property "Footprint" "M2SmartHomeFootprints:C_0402"
 			(at 256.54 41.91 0)
 			(effects
@@
 			)
 		)
-		(property "Footprint" "C_100n_0402:C_0402_1005Metric"
+		(property "Footprint" "M2SmartHomeFootprints:C_0402"
 			(at 236.22 41.91 0)
 			(effects
@@
 			)
 		)
-		(property "Footprint" "CONMHF1-SMD-T:LINX_CONMHF1-SMD-T"
+		(property "Footprint" "M2SmartHomeFootprints:CONMHF1-SMD-T"
 			(at 234.95 109.22 0)
 			(effects
@@
 			)
 		)
-		(property "Datasheet" ""
+		(property "Datasheet" "https://www.mouser.pl/datasheet/2/418/9/ENG_DS_conmhf1_smd_g_t_ds_A1-3238757.pdf"
 			(at 234.95 109.22 0)
 			(effects
@@
 			)
 		)
-		(property "Footprint" "C_1uF_0402:C_0402_1005Metric"
+		(property "Footprint" "M2SmartHomeFootprints:C_0201"
 			(at 226.06 41.91 0)
 			(effects
@@
 			)
 		)
-		(property "Footprint" "C_1uF_0402:C_0402_1005Metric"
+		(property "Footprint" "M2SmartHomeFootprints:C_0201"
 			(at 266.7 41.91 0)
 			(effects
@@
 			)
 		)
-		(property "Footprint" "R_24k_0402:R_0402_1005Metric"
+		(property "Footprint" "M2SmartHomeFootprints:R_0402"
 			(at 179.07 74.93 0)
 			(effects
@@
 			)
 		)
-		(property "Footprint" "R_10k_0402:R_0402_1005Metric"
+		(property "Footprint" "M2SmartHomeFootprints:R_0402"
 			(at 215.9 81.28 0)
 			(effects
@@
 			)
 		)
-		(property "Footprint" "C_100n_0402:C_0402_1005Metric"
+		(property "Footprint" "M2SmartHomeFootprints:C_0402"
 			(at 163.83 69.85 0)
 			(effects
@@
 			)
 		)
-		(property "Footprint" "R_500R_0402:R_0402_1005Metric"
+		(property "Footprint" "M2SmartHomeFootprints:R_0402"
 			(at 119.38 119.38 0)
 			(effects

Commit message: [#13] BRD fix 0201 coils
Parts:
- L4: footprint L_2n1_0201:L_0201_0603Metric -> M2SmartHomeFootprints:L_0201_0603Metric
Changed lines of the file:
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@@
 			)
 		)
-		(property "Footprint" "L_2n1_0201:L_0201_0603Metric"
+		(property "Footprint" "M2SmartHomeFootprints:L_0201_0603Metric"
 			(at 200.66 121.92 0)
 			(effects

Commit message: [#13] WIP Placement wifi
Parts:
- C55, C57, C75, C77: footprint M2SmartHomeFootprints:C_0201 -> M2SmartHomeFootprints:C_0402
Changed lines of the file:
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@@
 			)
 		)
-		(property "Footprint" "M2SmartHomeFootprints:C_0201"
+		(property "Footprint" "M2SmartHomeFootprints:C_0402"
 			(at 163.83 78.74 0)
 			(effects
@@
 			)
 		)
-		(property "Footprint" "M2SmartHomeFootprints:C_0201"
+		(property "Footprint" "M2SmartHomeFootprints:C_0402"
 			(at 246.38 41.91 0)
 			(effects
@@
 			)
 		)
-		(property "Footprint" "M2SmartHomeFootprints:C_0201"
+		(property "Footprint" "M2SmartHomeFootprints:C_0402"
 			(at 226.06 41.91 0)
 			(effects
@@
 			)
 		)
-		(property "Footprint" "M2SmartHomeFootprints:C_0201"
+		(property "Footprint" "M2SmartHomeFootprints:C_0402"
 			(at 266.7 41.91 0)
 			(effects
